File: board/rev-0/power.kicad_sch (KiCad schematic)
At the start: 0 parts

Commit message: Added power circuitry
Parts:
- added C23, C24, C29, C31: 4.7uF, symbol Device:C
- added C25, C30: 22uF, symbol Device:C
- added C26: 3.3nF, symbol Device:C
- added C27, C33: 0.1uF, symbol Device:C
- added C28, C32: 10uF, symbol Device:C
- added D19, D20: LED, symbol Device:LED
- added J8: S2B-PH-K-SLFSN, CONN_S2B-PH-K-S_JST, symbol my_lib:S2B-PH-K-SLFSN
- added L1: 2.2uH, symbol Device:L
- added R27, R30, R31: 10K, symbol Device:R_US
- added R28: 1.1K, symbol Device:R_US
- added R29: 1.13K, symbol Device:R_US
- added R32, R33: 1.5K, symbol Device:R_US
- added R34: 100K, symbol Device:R_US
- added U8: BQ24075RGT, Package_DFN_QFN:VQFN-16-1EP_3x3mm_P0.5mm_EP1.6x1.6mm, symbol Battery_Management:BQ24075RGT
- added U9: TPS62132, Package_DFN_QFN:VQFN-16-1EP_3x3mm_P0.5mm_EP1.68x1.68mm_ThermalVias, symbol Regulator_Switching:TPS62132
Connections:
- new net: C23.1, J8.2, U8.2 (BAT), U8.3 (BAT)
- new net: R29.1, U8.16 (ISET)
- new net: D19.2 (A), R32.2
- new net: L1.1, U9.1 (SW), U9.2 (SW), U9.3 (SW)
- new net: R28.1, U8.12 (ILIM)
- new net: C26.1, U9.9 (SS/TR)
- new net: R27.1, U8.1 (TS)
- new net: R34.2, U9.4 (PG)
- new net: D20.2 (A), R33.2
- new net GND: C23.2, C24.2, C25.2, C26.2, C27.2, C28.2, C29.2, C30.2, C31.2, C32.2, C33.2, J8.1, R27.2, R28.2, R29.2, R30.2, R31.2, U8.17 (VSS), U8.6 (EN1), U8.8 (VSS), U9.15 (GND), U9.16 (GND), U9.17 (GND), U9.5 (FB), U9.6 (GND), U9.7 (FSW), U9.8 (DEF)
- new net NCE: R31.1, U8.4 (~{CE})
- new net NCHG: D20.1 (K), U8.9 (~{CHG})
- new net NPGOOD: D19.1 (K), U8.7 (~{PGOOD})
- new net SW_OFF: R30.1, U8.15 (SYSOFF)
- new net VCC_3V3: C25.1, C31.1, C32.1, C33.1, L1.2, R34.1, U9.14 (VOS)
- new net VCC_5V5: C24.1, C27.1, C28.1, C29.1, C30.1, R32.1, R33.1, U8.10 (OUT), U8.11 (OUT), U8.5 (EN2), U9.10 (VIN), U9.11 (VIN), U9.12 (VIN), U9.13 (EN)
- new net VIN_5V: U8.13 (IN)
- no-connect marks 0 -> 1
