File: board/rev-0/biro-1-rev-0.kicad_pcb (KiCad board)
At the start: 4 copper layers, 158.5 x 81.5 mm, 134 parts, among them J1 I2C, J2 Conn_01x08, J3 USB_C_Receptacle_USB2.0_16P, J4 Conn_01x03, J5 Conn_01x03, J6 Conn_01x03, J7 Conn_01x03, J8 S2B-PH-K-SLFSN, U1 ESP32-S3-WROOM-1, U2 SN74LV1T34DBV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

Commit message: Added battery divider to ADC, created board step file, updated to kicad 9
Parts:
- turned R21 to 180 degrees
- turned R23 to 180 degrees
- turned R25 to 180 degrees
- turned R29 to 180 degrees
Routing:
- net /MCU/COL_0: track 0.00 -> 132.5 mm, vias 0 -> 1
- net /MCU/COL_1: track 0.00 -> 108.2 mm, vias 0 -> 1
- net /MCU/COL_2: track 0.00 -> 84.3 mm, vias 0 -> 1
- net /MCU/ROW_0: track 0.00 -> 78.6 mm, vias 0 -> 6
- net /MCU/ROW_2: track 0.00 -> 72.4 mm, vias 0 -> 6
- net /MCU/ROW_1: track 0.00 -> 57.0 mm, vias 0 -> 6
- net Net-(D1-A): track 0.00 -> 17.9 mm
- net Net-(D3-A): track 0.00 -> 17.8 mm
- net Net-(D5-A): track 0.00 -> 17.8 mm
- net Net-(D2-A): track 0.00 -> 17.8 mm
- net Net-(D4-A): track 0.00 -> 17.5 mm
- net Net-(D7-A): track 0.00 -> 17.5 mm
- net Net-(D9-A): track 0.00 -> 17.5 mm
- net Net-(D6-A): track 0.00 -> 17.4 mm
- net Net-(D8-A): track 0.00 -> 17.4 mm
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
Commit message: Added mounting holes, minor schematic fixes, layout progress
Parts:
- added J9: Conn_01x03, Connector_Wire:SolderWire-2sqmm_1x03_P7.8mm_D2mm_OD3.9mm, F.Cu at (190.2, 55.5)
- added R37: 100K, Resistor_SMD:R_0603_1608Metric, F.Cu at (209.8, 123.0)
- added R38: 50K, Resistor_SMD:R_0603_1608Metric, F.Cu at (209.8, 121.5)
- C11: value 330pF -> 0.1uF
- moved C11 5.07 mm to (209.8, 126.0), turned to 180 degrees
- moved C12 1.25 mm to (209.8, 124.5)
- moved R10 1.07 mm to (209.7, 120.0)
- moved R9 1.07 mm to (209.7, 118.5)
- moved C8 1.07 mm to (209.8, 117.0)
- turned R19 to 180 degrees
Connections:
- net Net-(C23-Pad1) renamed BAT+
- C11 pad 1: Net-(U5-VIN2N) -> Net-(U5-VIN2P)
- C11 pad 2: Net-(U5-VIN2P) -> GND
- U5 pad 4: Net-(U5-VIN2N) -> GND
Routing:
- net GND: track 0.00 -> 112.5 mm, vias 0 -> 79
- net VCC_5V5: track 4.47 -> 57.5 mm, vias 0 -> 43
- net VCC_3V3: track 0.00 -> 30.3 mm, vias 0 -> 24
- net VIN_5V: track 0.00 -> 4.71 mm, vias 0 -> 3
- net BAT+: track 0.00 -> 3.33 mm, vias 0 -> 2
- net Net-(U5-AVDD/LDO): track 0.00 -> 1.50 mm
- added copper zone on In2.Cu, net BAT+
- added copper zone on In2.Cu, net VCC_3V3
- added copper zone on In2.Cu, net VCC_5V5
- added copper zone on In2.Cu, net VIN_5V
