File: board/rev-0/mcu.kicad_sch (KiCad schematic)
At the start: 61 parts, among them J1 I2C, J2 Conn_01x08, J3 USB_C_Receptacle_USB2.0_16P, J4 Conn_01x03, J5 Conn_01x03, J6 Conn_01x03, J7 Conn_01x03, U1 ESP32-S3-WROOM-1, U7 SN74LV1T34DBV

Commit message: Added battery divider to ADC, created board step file, updated to kicad 9
Changed lines of the file:
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@@
 (kicad_sch
-	(version 20231120)
+	(version 20250114)
 	(generator "eeschema")
-	(generator_version "8.0")
+	(generator_version "9.0")
 	(paper "C")
 	(title_block
